File: pnp/pcb/mobo/motor_control.sch (KiCad schematic (older format))
At the start: 43 parts, among them J1 X_MOTOR, J2 Y_MOTOR1, J3 Z_MOTOR, J37 P_MOTOR, J38 C_MOTOR, J4 R_MOTOR, J48 Y_MOTOR2

Commit message: made XH THT-SMD footprints for connectors
Parts:
- J1: footprint Connector_JST:JST_XH_B4B-XH-A_1x04_P2.50mm_Vertical -> index:XH_4_THT-SMD
- JP1, JP10, JP11, JP12, JP13, JP14, JP15, JP16, JP17, JP18, JP19, JP2, JP20, JP21, JP22, JP23, JP24, JP3, JP4, JP5, JP6, JP7, JP8, JP9: footprint Connector_PinHeader_2.54mm:PinHeader_1x03_P2.54mm_Vertical -> Jumper:SolderJumper-3_P1.3mm_Open_RoundedPad1.0x1.5mm
Changed lines of the file:
@@
 F 0 "J1" H 3097 2182 50  0000 R CNN
 F 1 "X_MOTOR" H 3097 2273 50  0000 R CNN
-F 2 "Connector_JST:JST_XH_B4B-XH-A_1x04_P2.50mm_Vertical" H 3125 2300 50  0001 C CNN
+F 2 "index:XH_4_THT-SMD" H 3125 2300 50  0001 C CNN
 F 3 "~" H 3125 2300 50  0001 C CNN
 	1    3125 2300
@@
 F 0 "JP1" H 10050 1500 50  0000 C CNN
 F 1 "SolderJumper_3_Open" H 9400 1500 50  0000 C CNN
-F 2 "Connector_PinHeader_2.54mm:PinHeader_1x03_P2.54mm_Vertical" H 9900 1450 50  0001 C CNN
+F 2 "Jumper:SolderJumper-3_P1.3mm_Open_RoundedPad1.0x1.5mm" H 9900 1450 50  0001 C CNN
 F 3 "~" H 9900 1450 50  0001 C CNN
 	1    9900 1450
@@
 F 0 "JP2" H 10050 1800 50  0000 C CNN
 F 1 "SolderJumper_3_Open" H 9400 1800 50  0000 C CNN
-F 2 "Connector_PinHeader_2.54mm:PinHeader_1x03_P2.54mm_Vertical" H 9900 1750 50  0001 C CNN
+F 2 "Jumper:SolderJumper-3_P1.3mm_Open_RoundedPad1.0x1.5mm" H 9900 1750 50  0001 C CNN
 F 3 "~" H 9900 1750 50  0001 C CNN
 	1    9900 1750
@@
 F 0 "JP3" H 10050 2100 50  0000 C CNN
 F 1 "SolderJumper_3_Open" H 9400 2100 50  0000 C CNN
-F 2 "Connector_PinHeader_2.54mm:PinHeader_1x03_P2.54mm_Vertical" H 9900 2050 50  0001 C CNN
+F 2 "Jumper:SolderJumper-3_P1.3mm_Open_RoundedPad1.0x1.5mm" H 9900 2050 50  0001 C CNN
 F 3 "~" H 9900 2050 50  0001 C CNN
 	1    9900 2050
@@
 F 0 "JP4" H 10050 2400 50  0000 C CNN
 F 1 "SolderJumper_3_Open" H 9400 2400 50  0000 C CNN
-F 2 "Connector_PinHeader_2.54mm:PinHeader_1x03_P2.54mm_Vertical" H 9900 2350 50  0001 C CNN
+F 2 "Jumper:SolderJumper-3_P1.3mm_Open_RoundedPad1.0x1.5mm" H 9900 2350 50  0001 C CNN
 F 3 "~" H 9900 2350 50  0001 C CNN
 	1    9900 2350
@@
 F 0 "JP5" H 10075 2700 50  0000 C CNN
 F 1 "SolderJumper_3_Open" H 9375 2700 50  0000 C CNN
-F 2 "Connector_PinHeader_2.54mm:PinHeader_1x03_P2.54mm_Vertical" H 9900 2650 50  0001 C CNN
+F 2 "Jumper:SolderJumper-3_P1.3mm_Open_RoundedPad1.0x1.5mm" H 9900 2650 50  0001 C CNN
 F 3 "~" H 9900 2650 50  0001 C CNN
 	1    9900 2650
@@
 F 0 "JP6" H 10075 3000 50  0000 C CNN
 F 1 "SolderJumper_3_Open" H 9375 3000 50  0000 C CNN
-F 2 "Connector_PinHeader_2.54mm:PinHeader_1x03_P2.54mm_Vertical" H 9900 2950 50  0001 C CNN
+F 2 "Jumper:SolderJumper-3_P1.3mm_Open_RoundedPad1.0x1.5mm" H 9900 2950 50  0001 C CNN
 F 3 "~" H 9900 2950 50  0001 C CNN
 	1    9900 2950
@@
 F 0 "JP7" H 10075 3300 50  0000 C CNN
 F 1 "SolderJumper_3_Open" H 9375 3300 50  0000 C CNN
-F 2 "Connector_PinHeader_2.54mm:PinHeader_1x03_P2.54mm_Vertical" H 9900 3250 50  0001 C CNN
+F 2 "Jumper:SolderJumper-3_P1.3mm_Open_RoundedPad1.0x1.5mm" H 9900 3250 50  0001 C CNN
 F 3 "~" H 9900 3250 50  0001 C CNN
 	1    9900 3250
@@
 F 0 "JP8" H 10075 3600 50  0000 C CNN
 F 1 "SolderJumper_3_Open" H 9375 3600 50  0000 C CNN
-F 2 "Connector_PinHeader_2.54mm:PinHeader_1x03_P2.54mm_Vertical" H 9900 3550 50  0001 C CNN
+F 2 "Jumper:SolderJumper-3_P1.3mm_Open_RoundedPad1.0x1.5mm" H 9900 3550 50  0001 C CNN
 F 3 "~" H 9900 3550 50  0001 C CNN
 	1    9900 3550
@@
 F 0 "JP9" H 10075 3900 50  0000 C CNN
 F 1 "SolderJumper_3_Open" H 9375 3900 50  0000 C CNN
-F 2 "Connector_PinHeader_2.54mm:PinHeader_1x03_P2.54mm_Vertical" H 9900 3850 50  0001 C CNN
+F 2 "Jumper:SolderJumper-3_P1.3mm_Open_RoundedPad1.0x1.5mm" H 9900 3850 50  0001 C CNN
 F 3 "~" H 9900 3850 50  0001 C CNN
 	1    9900 3850
@@
 F 0 "JP10" H 10075 4200 50  0000 C CNN
 F 1 "SolderJumper_3_Open" H 9375 4200 50  0000 C CNN
-F 2 "Connector_PinHeader_2.54mm:PinHeader_1x03_P2.54mm_Vertical" H 9900 4150 50  0001 C CNN
+F 2 "Jumper:SolderJumper-3_P1.3mm_Open_RoundedPad1.0x1.5mm" H 9900 4150 50  0001 C CNN
 F 3 "~" H 9900 4150 50  0001 C CNN
 	1    9900 4150
@@
 F 0 "JP11" H 10075 4500 50  0000 C CNN
 F 1 "SolderJumper_3_Open" H 9375 4500 50  0000 C CNN
-F 2 "Connector_PinHeader_2.54mm:PinHeader_1x03_P2.54mm_Vertical" H 9900 4450 50  0001 C CNN
+F 2 "Jumper:SolderJumper-3_P1.3mm_Open_RoundedPad1.0x1.5mm" H 9900 4450 50  0001 C CNN
 F 3 "~" H 9900 4450 50  0001 C CNN
 	1    9900 4450
@@
 F 0 "JP12" H 10075 4800 50  0000 C CNN
 F 1 "SolderJumper_3_Open" H 9375 4800 50  0000 C CNN
-F 2 "Connector_PinHeader_2.54mm:PinHeader_1x03_P2.54mm_Vertical" H 9900 4750 50  0001 C CNN
+F 2 "Jumper:SolderJumper-3_P1.3mm_Open_RoundedPad1.0x1.5mm" H 9900 4750 50  0001 C CNN
 F 3 "~" H 9900 4750 50  0001 C CNN
 	1    9900 4750
@@
 F 0 "JP13" H 8050 1500 50  0000 C CNN
 F 1 "SolderJumper_3_Open" H 7400 1500 50  0000 C CNN
-F 2 "Connector_PinHeader_2.54mm:PinHeader_1x03_P2.54mm_Vertical" H 7900 1450 50  0001 C CNN
+F 2 "Jumper:SolderJumper-3_P1.3mm_Open_RoundedPad1.0x1.5mm" H 7900 1450 50  0001 C CNN
 F 3 "~" H 7900 1450 50  0001 C CNN
 	1    7900 1450
@@
 F 0 "JP14" H 8050 1800 50  0000 C CNN
 F 1 "SolderJumper_3_Open" H 7400 1800 50  0000 C CNN
-F 2 "Connector_PinHeader_2.54mm:PinHeader_1x03_P2.54mm_Vertical" H 7900 1750 50  0001 C CNN
+F 2 "Jumper:SolderJumper-3_P1.3mm_Open_RoundedPad1.0x1.5mm" H 7900 1750 50  0001 C CNN
 F 3 "~" H 7900 1750 50  0001 C CNN
 	1    7900 1750
@@
 F 0 "JP15" H 8050 2100 50  0000 C CNN
 F 1 "SolderJumper_3_Open" H 7400 2100 50  0000 C CNN
-F 2 "Connector_PinHeader_2.54mm:PinHeader_1x03_P2.54mm_Vertical" H 7900 2050 50  0001 C CNN
+F 2 "Jumper:SolderJumper-3_P1.3mm_Open_RoundedPad1.0x1.5mm" H 7900 2050 50  0001 C CNN
 F 3 "~" H 7900 2050 50  0001 C CNN
 	1    7900 2050
@@
 F 0 "JP16" H 8050 2400 50  0000 C CNN
 F 1 "SolderJumper_3_Open" H 7400 2400 50  0000 C CNN
-F 2 "Connector_PinHeader_2.54mm:PinHeader_1x03_P2.54mm_Vertical" H 7900 2350 50  0001 C CNN
+F 2 "Jumper:SolderJumper-3_P1.3mm_Open_RoundedPad1.0x1.5mm" H 7900 2350 50  0001 C CNN
 F 3 "~" H 7900 2350 50  0001 C CNN
 	1    7900 2350
@@
 F 0 "JP17" H 8075 2700 50  0000 C CNN
 F 1 "SolderJumper_3_Open" H 7375 2700 50  0000 C CNN
-F 2 "Connector_PinHeader_2.54mm:PinHeader_1x03_P2.54mm_Vertical" H 7900 2650 50  0001 C CNN
+F 2 "Jumper:SolderJumper-3_P1.3mm_Open_RoundedPad1.0x1.5mm" H 7900 2650 50  0001 C CNN
 F 3 "~" H 7900 2650 50  0001 C CNN
 	1    7900 2650
@@
 F 0 "JP18" H 8075 3000 50  0000 C CNN
 F 1 "SolderJumper_3_Open" H 7375 3000 50  0000 C CNN
-F 2 "Connector_PinHeader_2.54mm:PinHeader_1x03_P2.54mm_Vertical" H 7900 2950 50  0001 C CNN
+F 2 "Jumper:SolderJumper-3_P1.3mm_Open_RoundedPad1.0x1.5mm" H 7900 2950 50  0001 C CNN
 F 3 "~" H 7900 2950 50  0001 C CNN
 	1    7900 2950
@@
 F 0 "JP20" H 8075 3600 50  0000 C CNN
 F 1 "SolderJumper_3_Open" H 7375 3600 50  0000 C CNN
-F 2 "Connector_PinHeader_2.54mm:PinHeader_1x03_P2.54mm_Vertical" H 7900 3550 50  0001 C CNN
+F 2 "Jumper:SolderJumper-3_P1.3mm_Open_RoundedPad1.0x1.5mm" H 7900 3550 50  0001 C CNN
 F 3 "~" H 7900 3550 50  0001 C CNN
 	1    7900 3550
@@
 F 0 "JP21" H 8075 3900 50  0000 C CNN
 F 1 "SolderJumper_3_Open" H 7375 3900 50  0000 C CNN
-F 2 "Connector_PinHeader_2.54mm:PinHeader_1x03_P2.54mm_Vertical" H 7900 3850 50  0001 C CNN
+F 2 "Jumper:SolderJumper-3_P1.3mm_Open_RoundedPad1.0x1.5mm" H 7900 3850 50  0001 C CNN
 F 3 "~" H 7900 3850 50  0001 C CNN
 	1    7900 3850
@@
 F 0 "JP22" H 8075 4200 50  0000 C CNN
 F 1 "SolderJumper_3_Open" H 7375 4200 50  0000 C CNN
-F 2 "Connector_PinHeader_2.54mm:PinHeader_1x03_P2.54mm_Vertical" H 7900 4150 50  0001 C CNN
+F 2 "Jumper:SolderJumper-3_P1.3mm_Open_RoundedPad1.0x1.5mm" H 7900 4150 50  0001 C CNN
 F 3 "~" H 7900 4150 50  0001 C CNN
 	1    7900 4150
@@
 F 0 "JP23" H 8075 4500 50  0000 C CNN
 F 1 "SolderJumper_3_Open" H 7375 4500 50  0000 C CNN
-F 2 "Connector_PinHeader_2.54mm:PinHeader_1x03_P2.54mm_Vertical" H 7900 4450 50  0001 C CNN
+F 2 "Jumper:SolderJumper-3_P1.3mm_Open_RoundedPad1.0x1.5mm" H 7900 4450 50  0001 C CNN
 F 3 "~" H 7900 4450 50  0001 C CNN
 	1    7900 4450
@@
 F 0 "JP24" H 8075 4800 50  0000 C CNN
 F 1 "SolderJumper_3_Open" H 7375 4800 50  0000 C CNN
-F 2 "Connector_PinHeader_2.54mm:PinHeader_1x03_P2.54mm_Vertical" H 7900 4750 50  0001 C CNN
+F 2 "Jumper:SolderJumper-3_P1.3mm_Open_RoundedPad1.0x1.5mm" H 7900 4750 50  0001 C CNN
 F 3 "~" H 7900 4750 50  0001 C CNN
 	1    7900 4750
@@
 F 0 "JP19" H 8075 3300 50  0000 C CNN
 F 1 "SolderJumper_3_Open" H 7375 3300 50  0000 C CNN
-F 2 "Connector_PinHeader_2.54mm:PinHeader_1x03_P2.54mm_Vertical" H 7900 3250 50  0001 C CNN
+F 2 "Jumper:SolderJumper-3_P1.3mm_Open_RoundedPad1.0x1.5mm" H 7900 3250 50  0001 C CNN
 F 3 "~" H 7900 3250 50  0001 C CNN
 	1    7900 3250

Commit message: added in custom symbols for most parts in vacuum circuit, rewired it with those symbols, redid footprint allocation for the board. ready for layout
Parts:
- J1: footprint index:XH_4_THT-SMD -> Connector_JST:JST_XH_B4B-XH-A_1x04_P2.50mm_Vertical
Changed lines of the file:
@@
 F 0 "J1" H 3097 2182 50  0000 R CNN
 F 1 "X_MOTOR" H 3097 2273 50  0000 R CNN
-F 2 "index:XH_4_THT-SMD" H 3125 2300 50  0001 C CNN
+F 2 "Connector_JST:JST_XH_B4B-XH-A_1x04_P2.50mm_Vertical" H 3125 2300 50  0001 C CNN
 F 3 "~" H 3125 2300 50  0001 C CNN
 	1    3125 2300

Commit message: added 12v routing to increase current allowed
Parts:
- J1, J2, J3, J37, J38, J4, J48: footprint Connector_JST:JST_XH_B4B-XH-A_1x04_P2.50mm_Vertical -> Connector_JST:JST_XH_B04B-XH-A_1x04_P2.50mm_Vertical
Changed lines of the file:
@@
 F 0 "J3" H 3172 6382 50  0000 R CNN
 F 1 "Z_MOTOR" H 3172 6473 50  0000 R CNN
-F 2 "Connector_JST:JST_XH_B4B-XH-A_1x04_P2.50mm_Vertical" H 3200 6500 50  0001 C CNN
+F 2 "Connector_JST:JST_XH_B04B-XH-A_1x04_P2.50mm_Vertical" H 3200 6500 50  0001 C CNN
 F 3 "~" H 3200 6500 50  0001 C CNN
 	1    3200 6500
@@
 F 0 "J1" H 3097 2182 50  0000 R CNN
 F 1 "X_MOTOR" H 3097 2273 50  0000 R CNN
-F 2 "Connector_JST:JST_XH_B4B-XH-A_1x04_P2.50mm_Vertical" H 3125 2300 50  0001 C CNN
+F 2 "Connector_JST:JST_XH_B04B-XH-A_1x04_P2.50mm_Vertical" H 3125 2300 50  0001 C CNN
 F 3 "~" H 3125 2300 50  0001 C CNN
 	1    3125 2300
@@
 F 0 "J38" H 5747 6357 50  0000 R CNN
 F 1 "C_MOTOR" H 5747 6448 50  0000 R CNN
-F 2 "Connector_JST:JST_XH_B4B-XH-A_1x04_P2.50mm_Vertical" H 5775 6475 50  0001 C CNN
+F 2 "Connector_JST:JST_XH_B04B-XH-A_1x04_P2.50mm_Vertical" H 5775 6475 50  0001 C CNN
 F 3 "~" H 5775 6475 50  0001 C CNN
 	1    5775 6475
@@
 F 0 "J4" H 5747 2157 50  0000 R CNN
 F 1 "R_MOTOR" H 5747 2248 50  0000 R CNN
-F 2 "Connector_JST:JST_XH_B4B-XH-A_1x04_P2.50mm_Vertical" H 5775 2275 50  0001 C CNN
+F 2 "Connector_JST:JST_XH_B04B-XH-A_1x04_P2.50mm_Vertical" H 5775 2275 50  0001 C CNN
 F 3 "~" H 5775 2275 50  0001 C CNN
 	1    5775 2275
@@
 F 0 "J37" H 5747 4307 50  0000 R CNN
 F 1 "P_MOTOR" H 5747 4398 50  0000 R CNN
-F 2 "Connector_JST:JST_XH_B4B-XH-A_1x04_P2.50mm_Vertical" H 5775 4425 50  0001 C CNN
+F 2 "Connector_JST:JST_XH_B04B-XH-A_1x04_P2.50mm_Vertical" H 5775 4425 50  0001 C CNN
 F 3 "~" H 5775 4425 50  0001 C CNN
 	1    5775 4425
@@
 F 0 "J2" H 3075 4625 50  0000 R CNN
 F 1 "Y_MOTOR1" H 2625 4150 50  0000 R CNN
-F 2 "Connector_JST:JST_XH_B4B-XH-A_1x04_P2.50mm_Vertical" H 2850 4450 50  0001 C CNN
+F 2 "Connector_JST:JST_XH_B04B-XH-A_1x04_P2.50mm_Vertical" H 2850 4450 50  0001 C CNN
 F 3 "~" H 2850 4450 50  0001 C CNN
 	1    2850 4450
@@
 F 0 "J48" H 3175 4100 50  0000 R CNN
 F 1 "Y_MOTOR2" H 2825 4550 50  0000 R CNN
-F 2 "Connector_JST:JST_XH_B4B-XH-A_1x04_P2.50mm_Vertical" H 3000 4350 50  0001 C CNN
+F 2 "Connector_JST:JST_XH_B04B-XH-A_1x04_P2.50mm_Vertical" H 3000 4350 50  0001 C CNN
 F 3 "~" H 3000 4350 50  0001 C CNN
 	1    3000 4350

Commit message: assigned stepper motor config jumpers to be 2.54 dupont jumpers and not solder selectable jumpers
Parts:
- JP1, JP10, JP11, JP12, JP13, JP14, JP15, JP16, JP17, JP18, JP19, JP2, JP20, JP21, JP22, JP23, JP24, JP3, JP4, JP5, JP6, JP7, JP8, JP9: footprint Jumper:SolderJumper-3_P1.3mm_Open_RoundedPad1.0x1.5mm -> Connector_PinSocket_2.54mm:PinSocket_1x03_P2.54mm_Vertical
Changed lines of the file:
@@
 F 0 "JP1" H 10050 1500 50  0000 C CNN
 F 1 "SolderJumper_3_Open" H 9400 1500 50  0000 C CNN
-F 2 "Jumper:SolderJumper-3_P1.3mm_Open_RoundedPad1.0x1.5mm" H 9900 1450 50  0001 C CNN
+F 2 "Connector_PinSocket_2.54mm:PinSocket_1x03_P2.54mm_Vertical" H 9900 1450 50  0001 C CNN
 F 3 "~" H 9900 1450 50  0001 C CNN
 	1    9900 1450
@@
 F 0 "JP2" H 10050 1800 50  0000 C CNN
 F 1 "SolderJumper_3_Open" H 9400 1800 50  0000 C CNN
-F 2 "Jumper:SolderJumper-3_P1.3mm_Open_RoundedPad1.0x1.5mm" H 9900 1750 50  0001 C CNN
+F 2 "Connector_PinSocket_2.54mm:PinSocket_1x03_P2.54mm_Vertical" H 9900 1750 50  0001 C CNN
 F 3 "~" H 9900 1750 50  0001 C CNN
 	1    9900 1750
@@
 F 0 "JP3" H 10050 2100 50  0000 C CNN
 F 1 "SolderJumper_3_Open" H 9400 2100 50  0000 C CNN
-F 2 "Jumper:SolderJumper-3_P1.3mm_Open_RoundedPad1.0x1.5mm" H 9900 2050 50  0001 C CNN
+F 2 "Connector_PinSocket_2.54mm:PinSocket_1x03_P2.54mm_Vertical" H 9900 2050 50  0001 C CNN
 F 3 "~" H 9900 2050 50  0001 C CNN
 	1    9900 2050
@@
 F 0 "JP4" H 10050 2400 50  0000 C CNN
 F 1 "SolderJumper_3_Open" H 9400 2400 50  0000 C CNN
-F 2 "Jumper:SolderJumper-3_P1.3mm_Open_RoundedPad1.0x1.5mm" H 9900 2350 50  0001 C CNN
+F 2 "Connector_PinSocket_2.54mm:PinSocket_1x03_P2.54mm_Vertical" H 9900 2350 50  0001 C CNN
 F 3 "~" H 9900 2350 50  0001 C CNN
 	1    9900 2350
@@
 F 0 "JP5" H 10075 2700 50  0000 C CNN
 F 1 "SolderJumper_3_Open" H 9375 2700 50  0000 C CNN
-F 2 "Jumper:SolderJumper-3_P1.3mm_Open_RoundedPad1.0x1.5mm" H 9900 2650 50  0001 C CNN
+F 2 "Connector_PinSocket_2.54mm:PinSocket_1x03_P2.54mm_Vertical" H 9900 2650 50  0001 C CNN
 F 3 "~" H 9900 2650 50  0001 C CNN
 	1    9900 2650
@@
 F 0 "JP6" H 10075 3000 50  0000 C CNN
 F 1 "SolderJumper_3_Open" H 9375 3000 50  0000 C CNN
-F 2 "Jumper:SolderJumper-3_P1.3mm_Open_RoundedPad1.0x1.5mm" H 9900 2950 50  0001 C CNN
+F 2 "Connector_PinSocket_2.54mm:PinSocket_1x03_P2.54mm_Vertical" H 9900 2950 50  0001 C CNN
 F 3 "~" H 9900 2950 50  0001 C CNN
 	1    9900 2950
@@
 F 0 "JP7" H 10075 3300 50  0000 C CNN
 F 1 "SolderJumper_3_Open" H 9375 3300 50  0000 C CNN
-F 2 "Jumper:SolderJumper-3_P1.3mm_Open_RoundedPad1.0x1.5mm" H 9900 3250 50  0001 C CNN
+F 2 "Connector_PinSocket_2.54mm:PinSocket_1x03_P2.54mm_Vertical" H 9900 3250 50  0001 C CNN
 F 3 "~" H 9900 3250 50  0001 C CNN
 	1    9900 3250
@@
 F 0 "JP8" H 10075 3600 50  0000 C CNN
 F 1 "SolderJumper_3_Open" H 9375 3600 50  0000 C CNN
-F 2 "Jumper:SolderJumper-3_P1.3mm_Open_RoundedPad1.0x1.5mm" H 9900 3550 50  0001 C CNN
+F 2 "Connector_PinSocket_2.54mm:PinSocket_1x03_P2.54mm_Vertical" H 9900 3550 50  0001 C CNN
 F 3 "~" H 9900 3550 50  0001 C CNN
 	1    9900 3550
@@
 F 0 "JP9" H 10075 3900 50  0000 C CNN
 F 1 "SolderJumper_3_Open" H 9375 3900 50  0000 C CNN
-F 2 "Jumper:SolderJumper-3_P1.3mm_Open_RoundedPad1.0x1.5mm" H 9900 3850 50  0001 C CNN
+F 2 "Connector_PinSocket_2.54mm:PinSocket_1x03_P2.54mm_Vertical" H 9900 3850 50  0001 C CNN
 F 3 "~" H 9900 3850 50  0001 C CNN
 	1    9900 3850
@@
 F 0 "JP10" H 10075 4200 50  0000 C CNN
 F 1 "SolderJumper_3_Open" H 9375 4200 50  0000 C CNN
-F 2 "Jumper:SolderJumper-3_P1.3mm_Open_RoundedPad1.0x1.5mm" H 9900 4150 50  0001 C CNN
+F 2 "Connector_PinSocket_2.54mm:PinSocket_1x03_P2.54mm_Vertical" H 9900 4150 50  0001 C CNN
 F 3 "~" H 9900 4150 50  0001 C CNN
 	1    9900 4150
@@
 F 0 "JP11" H 10075 4500 50  0000 C CNN
 F 1 "SolderJumper_3_Open" H 9375 4500 50  0000 C CNN
-F 2 "Jumper:SolderJumper-3_P1.3mm_Open_RoundedPad1.0x1.5mm" H 9900 4450 50  0001 C CNN
+F 2 "Connector_PinSocket_2.54mm:PinSocket_1x03_P2.54mm_Vertical" H 9900 4450 50  0001 C CNN
 F 3 "~" H 9900 4450 50  0001 C CNN
 	1    9900 4450
@@
 F 0 "JP12" H 10075 4800 50  0000 C CNN
 F 1 "SolderJumper_3_Open" H 9375 4800 50  0000 C CNN
-F 2 "Jumper:SolderJumper-3_P1.3mm_Open_RoundedPad1.0x1.5mm" H 9900 4750 50  0001 C CNN
+F 2 "Connector_PinSocket_2.54mm:PinSocket_1x03_P2.54mm_Vertical" H 9900 4750 50  0001 C CNN
 F 3 "~" H 9900 4750 50  0001 C CNN
 	1    9900 4750
@@
 F 0 "JP13" H 8050 1500 50  0000 C CNN
 F 1 "SolderJumper_3_Open" H 7400 1500 50  0000 C CNN
-F 2 "Jumper:SolderJumper-3_P1.3mm_Open_RoundedPad1.0x1.5mm" H 7900 1450 50  0001 C CNN
+F 2 "Connector_PinSocket_2.54mm:PinSocket_1x03_P2.54mm_Vertical" H 7900 1450 50  0001 C CNN
 F 3 "~" H 7900 1450 50  0001 C CNN
 	1    7900 1450
@@
 F 0 "JP14" H 8050 1800 50  0000 C CNN
 F 1 "SolderJumper_3_Open" H 7400 1800 50  0000 C CNN
-F 2 "Jumper:SolderJumper-3_P1.3mm_Open_RoundedPad1.0x1.5mm" H 7900 1750 50  0001 C CNN
+F 2 "Connector_PinSocket_2.54mm:PinSocket_1x03_P2.54mm_Vertical" H 7900 1750 50  0001 C CNN
 F 3 "~" H 7900 1750 50  0001 C CNN
 	1    7900 1750
@@
 F 0 "JP15" H 8050 2100 50  0000 C CNN
 F 1 "SolderJumper_3_Open" H 7400 2100 50  0000 C CNN
-F 2 "Jumper:SolderJumper-3_P1.3mm_Open_RoundedPad1.0x1.5mm" H 7900 2050 50  0001 C CNN
+F 2 "Connector_PinSocket_2.54mm:PinSocket_1x03_P2.54mm_Vertical" H 7900 2050 50  0001 C CNN
 F 3 "~" H 7900 2050 50  0001 C CNN
 	1    7900 2050
@@
 F 0 "JP16" H 8050 2400 50  0000 C CNN
 F 1 "SolderJumper_3_Open" H 7400 2400 50  0000 C CNN
-F 2 "Jumper:SolderJumper-3_P1.3mm_Open_RoundedPad1.0x1.5mm" H 7900 2350 50  0001 C CNN
+F 2 "Connector_PinSocket_2.54mm:PinSocket_1x03_P2.54mm_Vertical" H 7900 2350 50  0001 C CNN
 F 3 "~" H 7900 2350 50  0001 C CNN
 	1    7900 2350
@@
 F 0 "JP17" H 8075 2700 50  0000 C CNN
 F 1 "SolderJumper_3_Open" H 7375 2700 50  0000 C CNN
-F 2 "Jumper:SolderJumper-3_P1.3mm_Open_RoundedPad1.0x1.5mm" H 7900 2650 50  0001 C CNN
+F 2 "Connector_PinSocket_2.54mm:PinSocket_1x03_P2.54mm_Vertical" H 7900 2650 50  0001 C CNN
 F 3 "~" H 7900 2650 50  0001 C CNN
 	1    7900 2650
@@
 F 0 "JP18" H 8075 3000 50  0000 C CNN
 F 1 "SolderJumper_3_Open" H 7375 3000 50  0000 C CNN
-F 2 "Jumper:SolderJumper-3_P1.3mm_Open_RoundedPad1.0x1.5mm" H 7900 2950 50  0001 C CNN
+F 2 "Connector_PinSocket_2.54mm:PinSocket_1x03_P2.54mm_Vertical" H 7900 2950 50  0001 C CNN
 F 3 "~" H 7900 2950 50  0001 C CNN
 	1    7900 2950
@@
 F 0 "JP20" H 8075 3600 50  0000 C CNN
 F 1 "SolderJumper_3_Open" H 7375 3600 50  0000 C CNN
-F 2 "Jumper:SolderJumper-3_P1.3mm_Open_RoundedPad1.0x1.5mm" H 7900 3550 50  0001 C CNN
+F 2 "Connector_PinSocket_2.54mm:PinSocket_1x03_P2.54mm_Vertical" H 7900 3550 50  0001 C CNN
 F 3 "~" H 7900 3550 50  0001 C CNN
 	1    7900 3550
@@
 F 0 "JP21" H 8075 3900 50  0000 C CNN
 F 1 "SolderJumper_3_Open" H 7375 3900 50  0000 C CNN
-F 2 "Jumper:SolderJumper-3_P1.3mm_Open_RoundedPad1.0x1.5mm" H 7900 3850 50  0001 C CNN
+F 2 "Connector_PinSocket_2.54mm:PinSocket_1x03_P2.54mm_Vertical" H 7900 3850 50  0001 C CNN
 F 3 "~" H 7900 3850 50  0001 C CNN
 	1    7900 3850
@@
 F 0 "JP22" H 8075 4200 50  0000 C CNN
 F 1 "SolderJumper_3_Open" H 7375 4200 50  0000 C CNN
-F 2 "Jumper:SolderJumper-3_P1.3mm_Open_RoundedPad1.0x1.5mm" H 7900 4150 50  0001 C CNN
+F 2 "Connector_PinSocket_2.54mm:PinSocket_1x03_P2.54mm_Vertical" H 7900 4150 50  0001 C CNN
 F 3 "~" H 7900 4150 50  0001 C CNN
 	1    7900 4150
@@
 F 0 "JP23" H 8075 4500 50  0000 C CNN
 F 1 "SolderJumper_3_Open" H 7375 4500 50  0000 C CNN
-F 2 "Jumper:SolderJumper-3_P1.3mm_Open_RoundedPad1.0x1.5mm" H 7900 4450 50  0001 C CNN
+F 2 "Connector_PinSocket_2.54mm:PinSocket_1x03_P2.54mm_Vertical" H 7900 4450 50  0001 C CNN
 F 3 "~" H 7900 4450 50  0001 C CNN
 	1    7900 4450
@@
 F 0 "JP24" H 8075 4800 50  0000 C CNN
 F 1 "SolderJumper_3_Open" H 7375 4800 50  0000 C CNN
-F 2 "Jumper:SolderJumper-3_P1.3mm_Open_RoundedPad1.0x1.5mm" H 7900 4750 50  0001 C CNN
+F 2 "Connector_PinSocket_2.54mm:PinSocket_1x03_P2.54mm_Vertical" H 7900 4750 50  0001 C CNN
 F 3 "~" H 7900 4750 50  0001 C CNN
 	1    7900 4750
@@
 F 0 "JP19" H 8075 3300 50  0000 C CNN
 F 1 "SolderJumper_3_Open" H 7375 3300 50  0000 C CNN
-F 2 "Jumper:SolderJumper-3_P1.3mm_Open_RoundedPad1.0x1.5mm" H 7900 3250 50  0001 C CNN
+F 2 "Connector_PinSocket_2.54mm:PinSocket_1x03_P2.54mm_Vertical" H 7900 3250 50  0001 C CNN
 F 3 "~" H 7900 3250 50  0001 C CNN
 	1    7900 3250
