File: pnp/pcb/mobo/motor.sch (KiCad schematic (older format))
At the start: 8 parts, among them M1 Stepper_Motor

Commit message: updated part info that gets exported for fab for the 1k resistors by the stepper drivers. changed LCSC and JLCPCB part numbers to correct ones
Parts:
- R6: JLCPCB C17855 -> C17513; LCSC C322766 -> C17513
Changed lines of the file:
@@
 AR Path="/5EB0C248/6035AFD9/602B8E66" Ref="#PWR?"  Part="1"
 AR Path="/5EB0C248/6036900B/602B8E66" Ref="#PWR?"  Part="1"
-F 0 "#PWR055" H 4625 4300 50  0001 C CNN
+F 0 "#PWR025" H 4625 4300 50  0001 C CNN
 F 1 "GND" H 4630 4377 50  0000 C CNN
 F 2 "" H 4625 4550 50  0001 C CNN
@@
 AR Path="/5EB0C248/6035AFD9/602B8E81" Ref="#PWR?"  Part="1"
 AR Path="/5EB0C248/6036900B/602B8E81" Ref="#PWR?"  Part="1"
-F 0 "#PWR054" H 4525 2900 50  0001 C CNN
+F 0 "#PWR024" H 4525 2900 50  0001 C CNN
 F 1 "+3V3" H 4540 3223 50  0000 C CNN
 F 2 "" H 4525 3050 50  0001 C CNN
@@
 AR Path="/5EB0C248/6035AFD9/602B8E8D" Ref="#PWR?"  Part="1"
 AR Path="/5EB0C248/6036900B/602B8E8D" Ref="#PWR?"  Part="1"
-F 0 "#PWR053" H 4125 3300 50  0001 C CNN
+F 0 "#PWR023" H 4125 3300 50  0001 C CNN
 F 1 "+3.3V" V 4140 3578 50  0000 L CNN
 F 2 "" H 4125 3450 50  0001 C CNN
@@
 AR Path="/5EB0C248/6035AFD9/602D9729" Ref="#PWR?"  Part="1"
 AR Path="/5EB0C248/6036900B/602D9729" Ref="#PWR?"  Part="1"
-F 0 "#PWR062" H 8225 3850 50  0001 C CNN
+F 0 "#PWR032" H 8225 3850 50  0001 C CNN
 F 1 "+3.3V" H 8240 4173 50  0000 C CNN
 F 2 "" H 8225 4000 50  0001 C CNN
@@
 AR Path="/5EB0C248/6035AFD9/602D973A" Ref="#PWR?"  Part="1"
 AR Path="/5EB0C248/6036900B/602D973A" Ref="#PWR?"  Part="1"
-F 0 "#PWR059" H 7175 3025 50  0001 C CNN
+F 0 "#PWR029" H 7175 3025 50  0001 C CNN
 F 1 "+3.3V" H 7190 3348 50  0000 C CNN
 F 2 "" H 7175 3175 50  0001 C CNN
@@
 AR Path="/5EB0C248/6035AFD9/602D9740" Ref="#PWR?"  Part="1"
 AR Path="/5EB0C248/6036900B/602D9740" Ref="#PWR?"  Part="1"
-F 0 "#PWR061" H 8225 3025 50  0001 C CNN
+F 0 "#PWR031" H 8225 3025 50  0001 C CNN
 F 1 "+3.3V" H 8240 3348 50  0000 C CNN
 F 2 "" H 8225 3175 50  0001 C CNN
@@
 AR Path="/5EB0C248/6035AFD9/602D9748" Ref="#PWR?"  Part="1"
 AR Path="/5EB0C248/6036900B/602D9748" Ref="#PWR?"  Part="1"
-F 0 "#PWR060" H 7175 3875 50  0001 C CNN
+F 0 "#PWR030" H 7175 3875 50  0001 C CNN
 F 1 "+3.3V" H 7190 4198 50  0000 C CNN
 F 2 "" H 7175 4025 50  0001 C CNN
@@
 AR Path="/5EB0C248/6035AFD9/603E21CF" Ref="#PWR?"  Part="1"
 AR Path="/5EB0C248/6036900B/603E21CF" Ref="#PWR?"  Part="1"
-F 0 "#PWR056" H 4725 2950 50  0001 C CNN
+F 0 "#PWR026" H 4725 2950 50  0001 C CNN
 F 1 "VDC" H 4740 3223 50  0000 C CNN
 F 2 "" H 4725 3050 50  0001 C CNN
@@
 AR Path="/5EB0C248/6035AFD9/604212D2" Ref="#PWR?"  Part="1"
 AR Path="/5EB0C248/6036900B/604212D2" Ref="#PWR?"  Part="1"
-F 0 "#PWR057" H 6050 2075 50  0001 C CNN
+F 0 "#PWR027" H 6050 2075 50  0001 C CNN
 F 1 "VDC" H 6065 2348 50  0000 C CNN
 F 2 "" H 6050 2175 50  0001 C CNN
@@
 AR Path="/5EB0C248/6035AFD9/604212D8" Ref="#PWR?"  Part="1"
 AR Path="/5EB0C248/6036900B/604212D8" Ref="#PWR?"  Part="1"
-F 0 "#PWR058" H 6050 2225 50  0001 C CNN
+F 0 "#PWR028" H 6050 2225 50  0001 C CNN
 F 1 "GND" H 6055 2302 50  0000 C CNN
 F 2 "" H 6050 2475 50  0001 C CNN
@@
 AR Path="/5EB0C248/6035AFD9/6040EB12" Ref="#FLG?"  Part="1"
 AR Path="/5EB0C248/6036900B/6040EB12" Ref="#FLG?"  Part="1"
-F 0 "#FLG015" H 8075 4275 50  0001 C CNN
+F 0 "#FLG06" H 8075 4275 50  0001 C CNN
 F 1 "PWR_FLAG" H 8075 4373 50  0001 C CNN
 F 2 "" H 8075 4200 50  0001 C CNN
@@
 AR Path="/5EB0C248/6035AFD9/6040EE3D" Ref="#FLG?"  Part="1"
 AR Path="/5EB0C248/6036900B/6040EE3D" Ref="#FLG?"  Part="1"
-F 0 "#FLG014" H 8075 3450 50  0001 C CNN
+F 0 "#FLG05" H 8075 3450 50  0001 C CNN
 F 1 "PWR_FLAG" H 8075 3548 50  0001 C CNN
 F 2 "" H 8075 3375 50  0001 C CNN
@@
 AR Path="/5EB0C248/6035AFD9/6040EFE9" Ref="#FLG?"  Part="1"
 AR Path="/5EB0C248/6036900B/6040EFE9" Ref="#FLG?"  Part="1"
-F 0 "#FLG013" H 7025 3450 50  0001 C CNN
+F 0 "#FLG04" H 7025 3450 50  0001 C CNN
 F 1 "PWR_FLAG" H 7025 3548 50  0001 C CNN
 F 2 "" H 7025 3375 50  0001 C CNN
@@
 F 3 "" H 3975 4250 50  0001 C CNN
 F 4 "" H 3975 4250 50  0001 C CNN "Digikey"
-F 5 "C17855" H 3975 4250 50  0001 C CNN "JLCPCB"
-F 6 "C322766" H 3975 4250 50  0001 C CNN "LCSC"
+F 5 "C17513" H 3975 4250 50  0001 C CNN "JLCPCB"
+F 6 "C17513" H 3975 4250 50  0001 C CNN "LCSC"
 F 7 "" H 3975 4250 50  0001 C CNN "Mouser"
 	1    3975 4250
