File: pnp/pcb/mobo/third_party_expansion.kicad_sch (KiCad schematic)
At the start: 20 parts, among them J5 AUX

Commit message: All pages checked
Parts:
- added L10: L_Ferrite_Small, Inductor_SMD:L_0805_2012Metric, symbol Device:L_Ferrite_Small
Connections:
- net VDC: now also L10.1; no longer J5.1 (Pin_1)
- new net: J5.1 (Pin_1), L10.2
Changed lines of the file:
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@@
+    (stroke (width 0) (type default))
+  )
+  (wire (pts (xy 87.63 49.53) (xy 96.52 49.53))
     (stroke (width 0) (type default))
   )
@@
   )
   (wire (pts (xy 81.28 52.07) (xy 82.55 52.07))
+    (stroke (width 0) (type default))
+  )
+  (wire (pts (xy 81.28 49.53) (xy 82.55 49.53))
     (stroke (width 0) (type default))
   )
@@
   )
   (symbol (lib_id "Device:L_Ferrite_Small") (at 85.09 52.07 90) (unit 1)
-    (in_bom yes) (on_board yes) (dnp no) (fields_autoplaced)
-    (property "Reference" "L18" (at 85.09 50.0921 90)
+    (in_bom yes) (on_board yes) (dnp no)
+    (property "Reference" "L18" (at 90.17 50.8 90)
       (effects (font (size 1.27 1.27)))
     )
@@
     )
   )
-  (symbol (lib_id "power:VDC") (at 96.52 49.53 90) (unit 1)
-    (in_bom yes) (on_board yes) (dnp no)
-    (property "Reference" "#PWR0129" (at 99.06 49.53 0)
-      (effects (font (size 1.27 1.27)) hide)
-    )
-    (property "Value" "VDC" (at 93.2942 49.149 90)
-      (effects (font (size 1.27 1.27)) (justify left))
-    )
-    (property "Footprint" "" (at 96.52 49.53 0)
-      (effects (font (size 1.27 1.27)) hide)
-    )
-    (property "Datasheet" "" (at 96.52 49.53 0)
+  (symbol (lib_id "power:VDC") (at 81.28 49.53 90) (unit 1)
+    (in_bom yes) (on_board yes) (dnp no)
+    (property "Reference" "#PWR0129" (at 83.82 49.53 0)
+      (effects (font (size 1.27 1.27)) hide)
+    )
+    (property "Value" "VDC" (at 78.0542 49.149 90)
+      (effects (font (size 1.27 1.27)) (justify left))
+    )
+    (property "Footprint" "" (at 81.28 49.53 0)
+      (effects (font (size 1.27 1.27)) hide)
+    )
+    (property "Datasheet" "" (at 81.28 49.53 0)
       (effects (font (size 1.27 1.27)) hide)
     )
@@
         )
       )
+    )
+  )
+  (symbol (lib_id "Device:L_Ferrite_Small") (at 85.09 49.53 90) (unit 1)
+    (in_bom yes) (on_board yes) (dnp no)
+    (property "Reference" "L10" (at 90.17 48.26 90)
+      (effects (font (size 1.27 1.27)))
+    )
+    (property "Value" "L_Ferrite_Small" (at 85.09 47.5521 90)
+      (effects (font (size 1.27 1.27)) hide)
+    )
+    (property "Footprint" "Inductor_SMD:L_0805_2012Metric" (at 85.09 49.53 0)
+      (effects (font (size 1.27 1.27)) hide)
+    )
+    (property "Datasheet" "~" (at 85.09 49.53 0)
+      (effects (font (size 1.27 1.27)) hide)
+    )
+    (pin "1")
+    (pin "2")
+    (instances
+      (project "mobo"
+        (path "/7255cbd1-8d38-4545-be9a-7fc5488ef942/00000000-0000-0000-0000-00005eb0c492"
+          (reference "L10") (unit 1)
+        )
+      )

Commit message: Mobo parts sourced
Parts:
- D17, D18, D19, D20, D21, D22, D23, D24, D25: JLCPCB (none) -> C2500; LCSC (none) -> C916421
- J5: JLCPCB (none) -> C9136
- L10, L18: JLCPCB (none) -> C1015; LCSC (none) -> C1015
- R11, R23, R35, R37, R38, R6, R7: value 100 -> 0; JLCPCB (none) -> C17477; LCSC (none) -> C17477
- R47: value 330 -> 0; JLCPCB (none) -> C17477; LCSC (none) -> C17477
- R48: value 510 -> 0; JLCPCB (none) -> C17477; LCSC (none) -> C17477
Changed lines of the file:
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@@
       (effects (font (size 0.75 0.75)))
     )
-    (property "Value" "100" (at 54.61 57.15 90)
+    (property "Value" "0" (at 54.61 57.15 90)
       (effects (font (size 0.75 0.75)))
     )
@@
       (effects (font (size 1.27 1.27)) hide)
     )
+    (property "JLCPCB" "C17477" (at 54.61 57.15 0)
+      (effects (font (size 1.27 1.27)) hide)
+    )
+    (property "LCSC" "C17477" (at 54.61 57.15 0)
+      (effects (font (size 1.27 1.27)) hide)
+    )
     (pin "1")
     (pin "2")
@@
       (effects (font (size 1.27 1.27)) hide)
     )
+    (property "JLCPCB" "C2500" (at 147.32 82.55 0)
+      (effects (font (size 1.27 1.27)) hide)
+    )
+    (property "LCSC" "C916421" (at 147.32 82.55 0)
+      (effects (font (size 1.27 1.27)) hide)
+    )
     (pin "1")
     (pin "2")
@@
       (effects (font (size 1.27 1.27)) hide)
     )
+    (property "JLCPCB" "C2500" (at 69.85 82.55 0)
+      (effects (font (size 1.27 1.27)) hide)
+    )
+    (property "LCSC" "C916421" (at 69.85 82.55 0)
+      (effects (font (size 1.27 1.27)) hide)
+    )
     (pin "1")
     (pin "2")
@@
       (effects (font (size 1.27 1.27)) hide)
     )
+    (property "JLCPCB" "C2500" (at 116.84 82.55 0)
+      (effects (font (size 1.27 1.27)) hide)
+    )
+    (property "LCSC" "C916421" (at 116.84 82.55 0)
+      (effects (font (size 1.27 1.27)) hide)
+    )
     (pin "1")
     (pin "2")
@@
       (effects (font (size 1.27 1.27)) hide)
     )
+    (property "JLCPCB" "C2500" (at 59.69 82.55 0)
+      (effects (font (size 1.27 1.27)) hide)
+    )
+    (property "LCSC" "C916421" (at 59.69 82.55 0)
+      (effects (font (size 1.27 1.27)) hide)
+    )
     (pin "1")
     (pin "2")
@@
       (effects (font (size 0.75 0.75)))
     )
-    (property "Value" "510" (at 161.29 62.23 90)
+    (property "Value" "0" (at 161.29 62.23 90)
       (effects (font (size 0.75 0.75)))
     )
@@
       (effects (font (size 1.27 1.27)) hide)
     )
+    (property "JLCPCB" "C17477" (at 161.29 62.23 0)
+      (effects (font (size 1.27 1.27)) hide)
+    )
+    (property "LCSC" "C17477" (at 161.29 62.23 0)
+      (effects (font (size 1.27 1.27)) hide)
+    )
     (pin "1")
     (pin "2")
@@
       (effects (font (size 0.75 0.75)))
     )
-    (property "Value" "100" (at 161.29 57.15 90)
+    (property "Value" "0" (at 161.29 57.15 90)
       (effects (font (size 0.75 0.75)))
     )
@@
       (effects (font (size 1.27 1.27)) hide)
     )
+    (property "JLCPCB" "C17477" (at 161.29 57.15 0)
+      (effects (font (size 1.27 1.27)) hide)
+    )
+    (property "LCSC" "C17477" (at 161.29 57.15 0)
+      (effects (font (size 1.27 1.27)) hide)
+    )
     (pin "1")
     (pin "2")
@@
       (effects (font (size 0.75 0.75)))
     )
-    (property "Value" "100" (at 54.61 62.23 90)
+    (property "Value" "0" (at 54.61 62.23 90)
       (effects (font (size 0.75 0.75)))
     )
@@
       (effects (font (size 1.27 1.27)) hide)
     )
+    (property "JLCPCB" "C17477" (at 54.61 62.23 0)
+      (effects (font (size 1.27 1.27)) hide)
+    )
+    (property "LCSC" "C17477" (at 54.61 62.23 0)
+      (effects (font (size 1.27 1.27)) hide)
+    )
     (pin "1")
     (pin "2")
@@
       (effects (font (size 1.27 1.27)) hide)
     )
+    (property "JLCPCB" "C2500" (at 127 82.55 0)
+      (effects (font (size 1.27 1.27)) hide)
+    )
+    (property "LCSC" "C916421" (at 127 82.55 0)
+      (effects (font (size 1.27 1.27)) hide)
+    )
     (pin "1")
     (pin "2")
@@
       (effects (font (size 0.75 0.75)))
     )
-    (property "Value" "100" (at 161.29 52.07 90)
+    (property "Value" "0" (at 161.29 52.07 90)
       (effects (font (size 0.75 0.75)))
     )
@@
       (effects (font (size 1.27 1.27)) hide)
     )
+    (property "JLCPCB" "C17477" (at 161.29 52.07 0)
+      (effects (font (size 1.27 1.27)) hide)
+    )
+    (property "LCSC" "C17477" (at 161.29 52.07 0)
+      (effects (font (size 1.27 1.27)) hide)
+    )
     (pin "1")
     (pin "2")
@@
       (effects (font (size 1.27 1.27)) hide)
     )
+    (property "JLCPCB" "C2500" (at 106.68 82.55 0)
+      (effects (font (size 1.27 1.27)) hide)
+    )
+    (property "LCSC" "C916421" (at 106.68 82.55 0)
+      (effects (font (size 1.27 1.27)) hide)
+    )
     (pin "1")
     (pin "2")
@@
     )
     (property "Datasheet" "~" (at 85.09 52.07 0)
+      (effects (font (size 1.27 1.27)) hide)
+    )
+    (property "JLCPCB" "C1015" (at 85.09 52.07 0)
+      (effects (font (size 1.27 1.27)) hide)
+    )
+    (property "LCSC" "C1015" (at 85.09 52.07 0)
       (effects (font (size 1.27 1.27)) hide)
     )
@@
       (effects (font (size 0.75 0.75)))
     )
-    (property "Value" "100" (at 161.29 54.61 90)
+    (property "Value" "0" (at 161.29 54.61 90)
       (effects (font (size 0.75 0.75)))
     )
@@
       (effects (font (size 1.27 1.27)) hide)
     )
+    (property "JLCPCB" "C17477" (at 161.29 54.61 0)
+      (effects (font (size 1.27 1.27)) hide)
+    )
+    (property "LCSC" "C17477" (at 161.29 54.61 0)
+      (effects (font (size 1.27 1.27)) hide)
+    )
     (pin "1")
     (pin "2")
@@
       (effects (font (size 1.27 1.27)) hide)
     )
+    (property "JLCPCB" "C2500" (at 137.16 82.55 0)
+      (effects (font (size 1.27 1.27)) hide)
+    )
+    (property "LCSC" "C916421" (at 137.16 82.55 0)
+      (effects (font (size 1.27 1.27)) hide)
+    )
     (pin "1")
     (pin "2")
@@
       (effects (font (size 0.75 0.75)))
     )
-    (property "Value" "100" (at 54.61 59.69 90)
+    (property "Value" "0" (at 54.61 59.69 90)
       (effects (font (size 0.75 0.75)))
     )
@@
       (effects (font (size 1.27 1.27)) hide)
     )
+    (property "JLCPCB" "C17477" (at 54.61 59.69 0)
+      (effects (font (size 1.27 1.27)) hide)
+    )
+    (property "LCSC" "C17477" (at 54.61 59.69 0)
+      (effects (font (size 1.27 1.27)) hide)
+    )
     (pin "1")
     (pin "2")
@@
     )
     (property "Datasheet" "https://assets.nexperia.com/documents/data-sheet/BAV99_SER.pdf" (at 80.01 82.55 0)
+      (effects (font (size 1.27 1.27)) hide)
+    )
+    (property "JLCPCB" "C2500" (at 80.01 82.55 0)
+      (effects (font (size 1.27 1.27)) hide)
+    )
+    (property "LCSC" "C916421" (at 80.01 82.55 0)
       (effects (font (size 1.27 1.27)) hide)
     )
@@
     )
     (property "LCSC" "C9136" (at 101.6 54.61 0)
+      (effects (font (size 1.27 1.27)) hide)
+    )
+    (property "JLCPCB" "C9136" (at 101.6 54.61 0)
       (effects (font (size 1.27 1.27)) hide)
     )
@@
       (effects (font (size 1.27 1.27)) hide)
     )
+    (property "JLCPCB" "C1015" (at 85.09 49.53 0)
+      (effects (font (size 1.27 1.27)) hide)
+    )
+    (property "LCSC" "C1015" (at 85.09 49.53 0)
+      (effects (font (size 1.27 1.27)) hide)
+    )
     (pin "1")
     (pin "2")
@@
       (effects (font (size 0.75 0.75)))
     )
-    (property "Value" "100" (at 54.61 54.61 90)
+    (property "Value" "0" (at 54.61 54.61 90)
       (effects (font (size 0.75 0.75)))
     )
@@
       (effects (font (size 1.27 1.27)) hide)
     )
+    (property "JLCPCB" "C17477" (at 54.61 54.61 0)
+      (effects (font (size 1.27 1.27)) hide)
+    )
+    (property "LCSC" "C17477" (at 54.61 54.61 0)
+      (effects (font (size 1.27 1.27)) hide)
+    )
     (pin "1")
     (pin "2")
@@
       (effects (font (size 0.75 0.75)))
     )
-    (property "Value" "330" (at 161.29 59.69 90)
+    (property "Value" "0" (at 161.29 59.69 90)
       (effects (font (size 0.75 0.75)))
     )
@@
       (effects (font (size 1.27 1.27)) hide)
     )
+    (property "JLCPCB" "C17477" (at 161.29 59.69 0)
+      (effects (font (size 1.27 1.27)) hide)
+    )
+    (property "LCSC" "C17477" (at 161.29 59.69 0)
+      (effects (font (size 1.27 1.27)) hide)
+    )
     (pin "1")
     (pin "2")
@@
       (effects (font (size 1.27 1.27)) hide)
     )
+    (property "JLCPCB" "C2500" (at 90.17 82.55 0)
+      (effects (font (size 1.27 1.27)) hide)
+    )
+    (property "LCSC" "C916421" (at 90.17 82.55 0)
+      (effects (font (size 1.27 1.27)) hide)
+    )
