File: pnp/pcb/mobo/RS485.kicad_sch (KiCad schematic)
At the start: 7 parts, among them J22 FEEDERS, U15 MAX3078E

Commit message: Capacitor sourcing
Parts:
- C121: LCSC C476766 -> C38141
- J22: JLCPCB (none) -> C67258; LCSC (none) -> C67258
Changed lines of the file:
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@@
 			(effects
 				(font
-					(size 1 1)
-					(color 223 129 255 1)
+					(size 1.27 1.27)
 				)
 				(hide yes)
@@
 			(effects
 				(font
-					(size 1 1)
-					(color 223 129 255 1)
-				)
-				(hide yes)
-			)
-		)
-		(property "Description" ""
+					(size 1.27 1.27)
+				)
+				(hide yes)
+			)
+		)
+		(property "Description" "test point"
 			(at 130.175 71.12 0)
 			(effects
@@
 			)
 		)
+		(property "JLCPCB" "C67258"
+			(at 151.765 66.04 0)
+			(effects
+				(font
+					(size 1.27 1.27)
+				)
+				(hide yes)
+			)
+		)
+		(property "LCSC" "C67258"
+			(at 151.765 66.04 0)
+			(effects
+				(font
+					(size 1.27 1.27)
+				)
+				(hide yes)
+			)
+		)
 		(pin "2"
 		)
@@
 			(effects
 				(font
-					(size 1 1)
-					(color 223 129 255 1)
+					(size 1.27 1.27)
 				)
 				(hide yes)
@@
 			(effects
 				(font
-					(size 1 1)
-					(color 223 129 255 1)
-				)
-				(hide yes)
-			)
-		)
-		(property "Description" ""
+					(size 1.27 1.27)
+				)
+				(hide yes)
+			)
+		)
+		(property "Description" "test point"
 			(at 130.175 53.34 0)
 			(effects
@@
 			)
 		)
-		(property "LCSC" "C476766"
+		(property "LCSC" "C38141"
 			(at 71.12 96.52 0)
 			(effects

Commit message: Sourcing complete
Parts:
- J22: LCSC C67258 -> C2829152
Changed lines of the file:
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@@
 			)
 		)
-		(property "LCSC" "C67258"
+		(property "LCSC" "C2829152"
 			(at 151.765 66.04 0)
 			(effects

Commit message: Sourcing of resistors complete
Parts:
- R58: JLCPCB C17437 -> C17414; LCSC C17437 -> C17414
Changed lines of the file:
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@@
 			)
 		)
-		(property "JLCPCB" "C17437"
+		(property "JLCPCB" "C17414"
 			(at 93.98 62.23 0)
 			(effects
@@
 			)
 		)
-		(property "LCSC" "C17437"
+		(property "LCSC" "C17414"
 			(at 93.98 62.23 0)
 			(effects

Commit message: Fix part sourcing
Parts:
- R58: JLCPCB C17414 -> C25280; LCSC C17414 -> C25280
Changed lines of the file:
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@@
 			)
 		)
-		(property "JLCPCB" "C17414"
+		(property "JLCPCB" "C25280"
 			(at 93.98 62.23 0)
 			(effects
@@
 			)
 		)
-		(property "LCSC" "C17414"
+		(property "LCSC" "C25280"
 			(at 93.98 62.23 0)
 			(effects

Commit message: Sourcing of ESD dodes
Parts:
- D27: JLCPCB (none) -> C521963; LCSC (none) -> C521963
Changed lines of the file:
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@@
+			)
+		)
+		(property "JLCPCB" "C521963"
+			(at 118.11 62.23 0)
+			(effects
+				(font
+					(size 1.27 1.27)
+				)
+				(hide yes)
+			)
+		)
+		(property "LCSC" "C521963"
+			(at 118.11 62.23 0)
+			(effects
+				(font
+					(size 1.27 1.27)
+				)
+				(hide yes)
 			)
 		)
