File: pnp/pcb/mobo/microcontroller.kicad_sch (KiCad schematic)
At the start: 56 parts, among them J11 XY_LIMIT, J13 HOST, J14 HACK_HEADER, J15 FAN, J17 Z_LIMIT, J2 SWD Header, Q5 AO3400A, Q6 AO3400A, SW1 SW_Push, SW2 SW_Push, U1 STM32F407VETx, U23 PESD5V2S2UT, U24 PESD3V3S2UT, U25 PESD3V3S2UT, U26 PESD3V3S2UT, U27 PESD3V3S2UT, Y1 8MHz

Commit message: Update RS485 to use THVD1400DR with split RC filter termination
Parts:
- renumbered C2 to C19, C6 to C20, C4 to C21, C7 to C22, C1 to C23, C16 to C24, C23 to C25, C17 to C26, C1 to C27, C3 to C28, C5 to C29, C8 to C30, C9 to C31, C29 to C32, C10 to C33, C11 to C34, C12 to C35, D9 to D10, D8 to D9, J13 to J2, J17 to J3, J11 to J4, J2 to J5, J14 to J6, J15 to J7, JP2 to JP1, Q5 to Q1, Q6 to Q2, R12 to R14, R57 to R15, R11 to R16, R59 to R17, R13 to R18, R14 to R19, R15 to R20, R16 to R21, R53 to R22, R8 to R23, R54 to R24, R55 to R25, R71 to R26, R56 to R27, U27 to U10, U24 to U5, U1 to U6, U23 to U7, U26 to U8, U25 to U9
