File: feeder/pcb/feederFloor/feederFloor.sch (KiCad schematic (older format))
At the start: 5 parts, among them J1 IDC, J2 Conn_01x10_Female, U1 DS2431

Commit message: Fixes #238.
Parts:
- J1: JLCPCB (none) -> C601936
- J2: Digikey 70AAJ-5-F0GCT-ND -> 70AAJ-5-M0GCT-ND; Mouser 652-70AAJ-5-F0G -> 652-70AAJ-5-M0G
Changed lines of the file:
@@
 F 2 "index:70AA-5" H 5600 1750 50  0001 C CNN
 F 3 "~" H 5600 1750 50  0001 C CNN
-F 4 "70AAJ-5-F0GCT-ND" V 5600 1750 50  0001 C CNN "Digikey"
-F 5 "652-70AAJ-5-F0G" V 5600 1750 50  0001 C CNN "Mouser"
+F 4 "70AAJ-5-M0GCT-ND" V 5600 1750 50  0001 C CNN "Digikey"
+F 5 "652-70AAJ-5-M0G" V 5600 1750 50  0001 C CNN "Mouser"
 	1    5600 1750
 	0    -1   -1   0
@@
 F 5 "710-61200621621" H 5550 3300 50  0001 C CNN "Mouser"
 F 6 "C601936" H 5550 3300 50  0001 C CNN "LCSC"
+F 7 "C601936" H 5550 3300 50  0001 C CNN "JLCPCB"
 	1    5550 3300
 	-1   0    0    1

Commit message: Route bus as diff pairs, pad for screw head and beautify
Parts:
- H1: footprint MountingHole:MountingHole_5.3mm_M5 -> MountingHole:MountingHole_5.3mm_M5_Pad_TopOnly
Connections:
- net labels added: RS-485+, RS-485-
- net labels removed: A, B
Changed lines of the file:
@@
 Text GLabel 6100 2450 2    50   Input ~ 0
 GND
-Text GLabel 5800 2150 2    50   Input ~ 0
-A
-Text GLabel 5900 2250 2    50   Input ~ 0
-B
 Text GLabel 5700 2050 2    50   Input ~ 0
 VIN
@@
 	4725 3300 4725 3800
 Connection ~ 4725 3300
-Text GLabel 5250 3200 0    50   Input ~ 0
-A
-Text GLabel 5750 3200 2    50   Input ~ 0
-B
 Text GLabel 6000 2350 2    50   Input ~ 0
 1WIRE
@@
 F 0 "H1" H 6900 2896 50  0000 L CNN
 F 1 "MountingHole" H 6900 2805 50  0000 L CNN
-F 2 "MountingHole:MountingHole_5.3mm_M5" H 6800 2850 50  0001 C CNN
+F 2 "MountingHole:MountingHole_5.3mm_M5_Pad_TopOnly" H 6800 2850 50  0001 C CNN
 F 3 "~" H 6800 2850 50  0001 C CNN
 	1    6800 2850
@@
 	1    0    0    -1
 $EndComp
+Text GLabel 6500 3650 2    50   Input ~ 0
+RS-485+
 Text GLabel 6500 3250 2    50   Input ~ 0
-B
-Text GLabel 6500 3650 2    50   Input ~ 0
-A
+RS-485-
 Wire Wire Line
 	6500 3250 6450 3250
@@
 Wire Wire Line
 	6450 3650 6500 3650
-Text Notes 6800 3425 0    50   ~ 0
+Text Notes 6800 3500 0    50   ~ 0
 R1 is a termination for the RS-485 bus. It must only \nbe installed on the final feeder floor in the chain.
 $Comp
@@
 Text GLabel 5750 3550 2    50   Input ~ 0
 GND
+Text GLabel 5250 3200 0    50   Input ~ 0
+RS-485+
+Text GLabel 5800 2150 2    50   Input ~ 0
+RS-485+
+Text GLabel 5750 3200 2    50   Input ~ 0
+RS-485-
+Text GLabel 5900 2250 2    50   Input ~ 0
+RS-485-
 $EndSCHEMATC

Commit message: Fix bus wires on feeder floors
Changed lines of the file:
@@
 Text GLabel 5750 3550 2    50   Input ~ 0
 GND
-Text GLabel 5250 3200 0    50   Input ~ 0
+Text GLabel 5750 3200 2    50   Input ~ 0
 RS-485+
 Text GLabel 5800 2150 2    50   Input ~ 0
 RS-485+
-Text GLabel 5750 3200 2    50   Input ~ 0
+Text GLabel 5250 3200 0    50   Input ~ 0
 RS-485-
 Text GLabel 5900 2250 2    50   Input ~ 0
