File: pnp/pcb/datum/datum.kicad_pcb (KiCad board)
At the start: 2 copper layers, 80 x 35 mm, 16 parts

Commit message: add missing component which was on the PCB but not on the schematic
Parts:
- FID1: renamed from REF**; value Fiducial_1mm_Mask2mm -> Fiducial
Changed lines of the file:
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@@
 			)
 		)
-		(property "Footprint" ""
+		(property "Footprint" "MountingHole:MountingHole_3.2mm_M3_Pad_Via"
 			(at 0 0 0)
 			(unlocked yes)
@@
 			)
 		)
-		(attr exclude_from_pos_files exclude_from_bom)
+		(property ki_fp_filters "MountingHole*Pad*")
+		(sheetname "Root")
+		(sheetfile "datum.kicad_sch")
+		(attr exclude_from_pos_files)
 		(fp_circle
 			(center 0 0)
@@
 			(remove_unused_layers no)
 			(net 1 "GND")
+			(pinfunction "1")
+			(pintype "input")
 		)
 		(pad "1" thru_hole circle
@@
 			(remove_unused_layers no)
 			(net 1 "GND")
+			(pinfunction "1")
+			(pintype "input")
 		)
 		(pad "1" thru_hole circle
@@
 			(remove_unused_layers no)
 			(net 1 "GND")
+			(pinfunction "1")
+			(pintype "input")
 		)
 		(pad "1" thru_hole circle
@@
 			(remove_unused_layers no)
 			(net 1 "GND")
+			(pinfunction "1")
+			(pintype "input")
 		)
 		(pad "1" thru_hole circle
@@
 			(remove_unused_layers no)
 			(net 1 "GND")
+			(pinfunction "1")
+			(pintype "input")
 		)
 		(pad "1" thru_hole circle
@@
 			(remove_unused_layers no)
 			(net 1 "GND")
+			(pinfunction "1")
+			(pintype "input")
 		)
 		(pad "1" thru_hole circle
@@
 			(remove_unused_layers no)
 			(net 1 "GND")
+			(pinfunction "1")
+			(pintype "input")
 		)
 		(pad "1" thru_hole circle
@@
 			(remove_unused_layers no)
 			(net 1 "GND")
+			(pinfunction "1")
+			(pintype "input")
 		)
 		(pad "1" thru_hole circle
@@
 			(remove_unused_layers no)
 			(net 1 "GND")
+			(pinfunction "1")
+			(pintype "input")
 		)
 	)
@@
 			)
 		)
-		(property "Footprint" ""
+		(property "Footprint" "MountingHole:MountingHole_3.2mm_M3_Pad_Via"
 			(at 0 0 0)
 			(unlocked yes)
@@
 			)
 		)
-		(attr exclude_from_pos_files exclude_from_bom)
+		(property ki_fp_filters "MountingHole*Pad*")
+		(sheetname "Root")
+		(sheetfile "datum.kicad_sch")
+		(attr exclude_from_pos_files)
 		(fp_circle
 			(center 0 0)
@@
 			(remove_unused_layers no)
 			(net 1 "GND")
+			(pinfunction "1")
+			(pintype "input")
 		)
 		(pad "1" thru_hole circle
@@
 			(remove_unused_layers no)
 			(net 1 "GND")
+			(pinfunction "1")
+			(pintype "input")
 		)
 		(pad "1" thru_hole circle
@@
 			(remove_unused_layers no)
 			(net 1 "GND")
+			(pinfunction "1")
+			(pintype "input")
 		)
 		(pad "1" thru_hole circle
@@
 			(remove_unused_layers no)
 			(net 1 "GND")
+			(pinfunction "1")
+			(pintype "input")
 		)
 		(pad "1" thru_hole circle
@@
 			(remove_unused_layers no)
 			(net 1 "GND")
+			(pinfunction "1")
+			(pintype "input")
 		)
 		(pad "1" thru_hole circle
@@
 			(remove_unused_layers no)
 			(net 1 "GND")
+			(pinfunction "1")
+			(pintype "input")
 		)
 		(pad "1" thru_hole circle
@@
 			(remove_unused_layers no)
 			(net 1 "GND")
+			(pinfunction "1")
+			(pintype "input")
 		)
 		(pad "1" thru_hole circle
@@
 			(remove_unused_layers no)
 			(net 1 "GND")
+			(pinfunction "1")
+			(pintype "input")
 		)
 		(pad "1" thru_hole circle
@@
 			(remove_unused_layers no)
 			(net 1 "GND")
+			(pinfunction "1")
+			(pintype "input")
 		)
 	)
@@
 			)
 		)
-		(property "Footprint" ""
+		(property "Footprint" "MountingHole:MountingHole_3.2mm_M3_Pad_Via"
 			(at 0 0 0)
 			(unlocked yes)
@@
 			)
 		)
-		(attr exclude_from_pos_files exclude_from_bom)
+		(property ki_fp_filters "MountingHole*Pad*")
+		(sheetname "Root")
+		(sheetfile "datum.kicad_sch")
+		(attr exclude_from_pos_files)
 		(fp_circle
 			(center 0 0)
@@
 			(remove_unused_layers no)
 			(net 1 "GND")
+			(pinfunction "1")
+			(pintype "input")
 		)
 		(pad "1" thru_hole circle
@@
 			(remove_unused_layers no)
 			(net 1 "GND")
+			(pinfunction "1")
+			(pintype "input")
 		)
 		(pad "1" thru_hole circle
@@
 			(remove_unused_layers no)
 			(net 1 "GND")
+			(pinfunction "1")
+			(pintype "input")
 		)
 		(pad "1" thru_hole circle
@@
 			(remove_unused_layers no)
 			(net 1 "GND")
+			(pinfunction "1")
+			(pintype "input")
 		)
 		(pad "1" thru_hole circle
@@
 			(remove_unused_layers no)
 			(net 1 "GND")
+			(pinfunction "1")
+			(pintype "input")
 		)
 		(pad "1" thru_hole circle
@@
 			(remove_unused_layers no)
 			(net 1 "GND")
+			(pinfunction "1")
+			(pintype "input")
 		)
 		(pad "1" thru_hole circle
@@
 			(remove_unused_layers no)
 			(net 1 "GND")
+			(pinfunction "1")
+			(pintype "input")
 		)
 		(pad "1" thru_hole circle
@@
 			(remove_unused_layers no)
 			(net 1 "GND")
+			(pinfunction "1")
+			(pintype "input")
 		)
 		(pad "1" thru_hole circle
@@
 			(remove_unused_layers no)
 			(net 1 "GND")
+			(pinfunction "1")
+			(pintype "input")
 		)
 	)
@@
 			)
 		)
-		(property "Footprint" ""
+		(property "Footprint" "MountingHole:MountingHole_3.2mm_M3_Pad_Via"
 			(at 0 0 0)
 			(unlocked yes)
@@
 			)
 		)
-		(attr exclude_from_pos_files exclude_from_bom)
+		(property ki_fp_filters "MountingHole*Pad*")
+		(sheetname "Root")
+		(sheetfile "datum.kicad_sch")
+		(attr exclude_from_pos_files)
 		(fp_circle
 			(center 0 0)
@@
 			(remove_unused_layers no)
 			(net 1 "GND")
+			(pinfunction "1")
+			(pintype "input")
 		)
 		(pad "1" thru_hole circle
@@
 			(remove_unused_layers no)
 			(net 1 "GND")
+			(pinfunction "1")
+			(pintype "input")
 		)
 		(pad "1" thru_hole circle
@@
 			(remove_unused_layers no)
 			(net 1 "GND")
+			(pinfunction "1")
+			(pintype "input")
 		)
 		(pad "1" thru_hole circle
@@
 			(remove_unused_layers no)
 			(net 1 "GND")
+			(pinfunction "1")
+			(pintype "input")
 		)
 		(pad "1" thru_hole circle
@@
 			(remove_unused_layers no)
 			(net 1 "GND")
+			(pinfunction "1")
+			(pintype "input")
 		)
 		(pad "1" thru_hole circle
@@
 			(remove_unused_layers no)
 			(net 1 "GND")
+			(pinfunction "1")
+			(pintype "input")
 		)
 		(pad "1" thru_hole circle
@@
 			(remove_unused_layers no)
 			(net 1 "GND")
+			(pinfunction "1")
+			(pintype "input")
 		)
 		(pad "1" thru_hole circle
@@
 			(remove_unused_layers no)
 			(net 1 "GND")
+			(pinfunction "1")
+			(pintype "input")
 		)
 		(pad "1" thru_hole circle
@@
 			(remove_unused_layers no)
 			(net 1 "GND")
+			(pinfunction "1")
+			(pintype "input")
 		)
 	)
@@
 		(descr "Circular Fiducial, 1mm bare copper, 2mm soldermask opening (Level A)")
 		(tags "fiducial")
-		(property "Reference" "REF**"
+		(property "Reference" "FID1"
 			(at 0 -2 0)
 			(layer "F.SilkS")
@@
 			)
 		)
-		(property "Value" "Fiducial_1mm_Mask2mm"
+		(property "Value" "Fiducial"
 			(at 0 2 0)
 			(layer "F.Fab")
@@
 			)
 		)
-		(property "Footprint" ""
+		(property "Footprint" "Fiducial:Fiducial_1mm_Mask2mm"
 			(at 0 0 0)
 			(unlocked yes)
@@
 			)
 		)
-		(property "Description" ""
+		(property "Description" "Fiducial Marker"
 			(at 0 0 0)
 			(unlocked yes)
@@
 			)
 		)
-		(attr smd)
+		(property ki_fp_filters "Fiducial*")
+		(sheetname "Root")
+		(sheetfile "datum.kicad_sch")
+		(attr smd exclude_from_bom)
 		(fp_circle
 			(center 0 0)
@@
 			)
 		)
-		(property "Footprint" ""
+		(property "Footprint" "TestPoint:TestPoint_Pad_D4.0mm"
 			(at 0 0 0)
 			(unlocked yes)
@@
 			)
 		)
-		(attr exclude_from_pos_files exclude_from_bom)
+		(property ki_fp_filters "Pin* Test*")
+		(sheetname "Root")
+		(sheetfile "datum.kicad_sch")
+		(attr exclude_from_pos_files)
 		(fp_circle
 			(center 0 0)
@@
 			(layers "B.Cu" "B.Mask")
 			(net 1 "GND")
+			(pinfunction "1")
+			(pintype "passive")
 		)
 	)
