File: pnp/pcb/datum/datum.kicad_pcb (KiCad board)
At the start: 2 copper layers, 80 x 35 mm, 16 parts

Commit message: Fix fiducial reference designators
Parts:
- FID2, FID3, FID4, FID5, FID6, FID7: renamed from REF**; value Fiducial_1mm_Mask3mm -> Fiducial
Changed lines of the file:
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@@
 		(descr "Circular Fiducial, 1mm bare copper, 3mm soldermask opening (recommended)")
 		(tags "fiducial")
-		(property "Reference" "REF**"
+		(property "Reference" "FID4"
 			(at 0 -2.54 0)
 			(layer "F.SilkS")
@@
 			)
 		)
-		(property "Value" "Fiducial_1mm_Mask3mm"
+		(property "Value" "Fiducial"
 			(at 0 2.286 0)
 			(layer "F.Fab")
@@
 			)
 		)
-		(property "Footprint" ""
+		(property "Footprint" "Fiducial:Fiducial_1mm_Mask3mm"
 			(at 0 0 0)
 			(unlocked yes)
@@
 			)
 		)
-		(property "Description" ""
-			(at 0 0 0)
-			(unlocked yes)
-			(layer "F.Fab")
-			(hide yes)
-			(effects
-				(font
-					(size 1.27 1.27)
-				)
-			)
-		)
-		(attr smd)
+		(property "Description" "Fiducial Marker"
+			(at 0 0 0)
+			(unlocked yes)
+			(layer "F.Fab")
+			(hide yes)
+			(effects
+				(font
+					(size 1.27 1.27)
+				)
+			)
+		)
+		(property ki_fp_filters "Fiducial*")
+		(sheetname "Root")
+		(sheetfile "datum.kicad_sch")
+		(attr smd exclude_from_bom)
 		(fp_circle
 			(center 0 0)
@@
 		(descr "Circular Fiducial, 1mm bare copper, 3mm soldermask opening (recommended)")
 		(tags "fiducial")
-		(property "Reference" "REF**"
+		(property "Reference" "FID2"
 			(at 0 -2.54 0)
 			(layer "F.SilkS")
@@
 			)
 		)
-		(property "Value" "Fiducial_1mm_Mask3mm"
+		(property "Value" "Fiducial"
 			(at 0 2.286 0)
 			(layer "F.Fab")
@@
 			)
 		)
-		(property "Footprint" ""
+		(property "Footprint" "Fiducial:Fiducial_1mm_Mask3mm"
 			(at 0 0 0)
 			(unlocked yes)
@@
 			)
 		)
-		(property "Description" ""
-			(at 0 0 0)
-			(unlocked yes)
-			(layer "F.Fab")
-			(hide yes)
-			(effects
-				(font
-					(size 1.27 1.27)
-				)
-			)
-		)
-		(attr smd)
+		(property "Description" "Fiducial Marker"
+			(at 0 0 0)
+			(unlocked yes)
+			(layer "F.Fab")
+			(hide yes)
+			(effects
+				(font
+					(size 1.27 1.27)
+				)
+			)
+		)
+		(property ki_fp_filters "Fiducial*")
+		(sheetname "Root")
+		(sheetfile "datum.kicad_sch")
+		(attr smd exclude_from_bom)
 		(fp_circle
 			(center 0 0)
@@
 		(descr "Circular Fiducial, 1mm bare copper, 3mm soldermask opening (recommended)")
 		(tags "fiducial")
-		(property "Reference" "REF**"
+		(property "Reference" "FID7"
 			(at 0 -2.54 0)
 			(layer "F.SilkS")
@@
 			)
 		)
-		(property "Value" "Fiducial_1mm_Mask3mm"
+		(property "Value" "Fiducial"
 			(at 0 2.286 0)
 			(layer "F.Fab")
@@
 			)
 		)
-		(property "Footprint" ""
+		(property "Footprint" "Fiducial:Fiducial_1mm_Mask3mm"
 			(at 0 0 0)
 			(unlocked yes)
@@
 			)
 		)
-		(property "Description" ""
-			(at 0 0 0)
-			(unlocked yes)
-			(layer "F.Fab")
-			(hide yes)
-			(effects
-				(font
-					(size 1.27 1.27)
-				)
-			)
-		)
-		(attr smd)
+		(property "Description" "Fiducial Marker"
+			(at 0 0 0)
+			(unlocked yes)
+			(layer "F.Fab")
+			(hide yes)
+			(effects
+				(font
+					(size 1.27 1.27)
+				)
+			)
+		)
+		(property ki_fp_filters "Fiducial*")
+		(sheetname "Root")
+		(sheetfile "datum.kicad_sch")
+		(attr smd exclude_from_bom)
 		(fp_circle
 			(center 0 0)
@@
 		(descr "Circular Fiducial, 1mm bare copper, 3mm soldermask opening (recommended)")
 		(tags "fiducial")
-		(property "Reference" "REF**"
+		(property "Reference" "FID6"
 			(at 0 -2.54 0)
 			(layer "F.SilkS")
@@
 			)
 		)
-		(property "Value" "Fiducial_1mm_Mask3mm"
+		(property "Value" "Fiducial"
 			(at 0 2.286 0)
 			(layer "F.Fab")
@@
 			)
 		)
-		(property "Footprint" ""
+		(property "Footprint" "Fiducial:Fiducial_1mm_Mask3mm"
 			(at 0 0 0)
 			(unlocked yes)
@@
 			)
 		)
-		(property "Description" ""
-			(at 0 0 0)
-			(unlocked yes)
-			(layer "F.Fab")
-			(hide yes)
-			(effects
-				(font
-					(size 1.27 1.27)
-				)
-			)
-		)
-		(attr smd)
+		(property "Description" "Fiducial Marker"
+			(at 0 0 0)
+			(unlocked yes)
+			(layer "F.Fab")
+			(hide yes)
+			(effects
+				(font
+					(size 1.27 1.27)
+				)
+			)
+		)
+		(property ki_fp_filters "Fiducial*")
+		(sheetname "Root")
+		(sheetfile "datum.kicad_sch")
+		(attr smd exclude_from_bom)
 		(fp_circle
 			(center 0 0)
@@
 		(descr "Circular Fiducial, 1mm bare copper, 3mm soldermask opening (recommended)")
 		(tags "fiducial")
-		(property "Reference" "REF**"
+		(property "Reference" "FID5"
 			(at 0 -2.54 0)
 			(layer "F.SilkS")
@@
 			)
 		)
-		(property "Value" "Fiducial_1mm_Mask3mm"
+		(property "Value" "Fiducial"
 			(at 0 2.286 0)
 			(layer "F.Fab")
@@
 			)
 		)
-		(property "Footprint" ""
+		(property "Footprint" "Fiducial:Fiducial_1mm_Mask3mm"
 			(at 0 0 0)
 			(unlocked yes)
@@
 			)
 		)
-		(property "Description" ""
-			(at 0 0 0)
-			(unlocked yes)
-			(layer "F.Fab")
-			(hide yes)
-			(effects
-				(font
-					(size 1.27 1.27)
-				)
-			)
-		)
-		(attr smd)
+		(property "Description" "Fiducial Marker"
+			(at 0 0 0)
+			(unlocked yes)
+			(layer "F.Fab")
+			(hide yes)
+			(effects
+				(font
+					(size 1.27 1.27)
+				)
+			)
+		)
+		(property ki_fp_filters "Fiducial*")
+		(sheetname "Root")
+		(sheetfile "datum.kicad_sch")
+		(attr smd exclude_from_bom)
 		(fp_circle
 			(center 0 0)
@@
 		(descr "Circular Fiducial, 1mm bare copper, 3mm soldermask opening (recommended)")
 		(tags "fiducial")
-		(property "Reference" "REF**"
+		(property "Reference" "FID3"
 			(at 0 -2.54 0)
 			(layer "F.SilkS")
@@
 			)
 		)
-		(property "Value" "Fiducial_1mm_Mask3mm"
+		(property "Value" "Fiducial"
 			(at 0 2.286 0)
 			(layer "F.Fab")
@@
 			)
 		)
-		(property "Footprint" ""
+		(property "Footprint" "Fiducial:Fiducial_1mm_Mask3mm"
 			(at 0 0 0)
 			(unlocked yes)
@@
 			)
 		)
-		(property "Description" ""
-			(at 0 0 0)
-			(unlocked yes)
-			(layer "F.Fab")
-			(hide yes)
-			(effects
-				(font
-					(size 1.27 1.27)
-				)
-			)
-		)
-		(attr smd)
+		(property "Description" "Fiducial Marker"
+			(at 0 0 0)
+			(unlocked yes)
+			(layer "F.Fab")
+			(hide yes)
+			(effects
+				(font
+					(size 1.27 1.27)
+				)
+			)
+		)
+		(property ki_fp_filters "Fiducial*")
+		(sheetname "Root")
+		(sheetfile "datum.kicad_sch")
+		(attr smd exclude_from_bom)
 		(fp_circle
 			(center 0 0)

Commit message: Fix datum ruler designator
Parts:
- renumbered REF** to G4
Changed lines of the file:
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@@
 		(layer "F.Cu")
 		(at 25 -10)
-		(property "Reference" "REF**"
+		(property "Reference" "G4"
 			(at 7.00024 -3.5005 0)
 			(layer "F.SilkS")
