File: feeder/pcb/mobo/mobo.kicad_sch (KiCad schematic)
At the start: 60 parts, among them J1 SWD_10, J2 FTDI_HEADER, J3 PLATED_PADS, M1 PEEL_MOTOR, M2 DRIVE_MOTOR, SW1 RESET, SW2 BUTTON_1, SW3 BUTTON_2, SW4 BOOT, U1 QRE1113GR, U2 STM32F103C8Tx, U3 TCS40DPR, U4 AP1117-33, U5 MCP16301, U6 DRV8833PWP, U7 MAX3078E, Y1 8MHz

Commit message: Add component PN to feeder pcb
Parts:
- SW1, SW2, SW3, SW4: JLCPCB (none) -> C128539
Changed lines of the file:
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@@
       (effects (font (size 1.27 1.27)) hide)
     )
-    (property "JLCPCB" "" (id 4) (at 103.505 130.175 0)
+    (property "JLCPCB" "C128539 " (id 4) (at 103.505 130.175 0)
       (effects (font (size 1.27 1.27)) hide)
     )
@@
       (effects (font (size 1.27 1.27)) hide)
     )
-    (property "JLCPCB" "" (id 4) (at 103.505 147.955 0)
+    (property "JLCPCB" "C128539 " (id 4) (at 103.505 147.955 0)
       (effects (font (size 1.27 1.27)) hide)
     )
@@
       (effects (font (size 1.27 1.27)) hide)
     )
-    (property "JLCPCB" "" (id 4) (at 49.53 24.13 90)
+    (property "JLCPCB" "C128539 " (id 4) (at 49.53 24.13 90)
       (effects (font (size 1.27 1.27)) hide)
     )
@@
       (effects (font (size 1.27 1.27)) hide)
     )
-    (property "JLCPCB" "" (id 4) (at 151.13 58.42 0)
-      (effects (font (size 1.27 1.27)) hide)
-    )
+    (property "JLCPCB" "C128539 " (id 4) (at 151.13 58.42 0)
+      (effects (font (size 1.27 1.27)) hide)
+    )
