File: pnp/pcb/ringLight/ringLight.kicad_sch (KiCad schematic)
At the start: 24 parts, among them J1 Connector Vertical, J2 Connector Horizontal, U1 74AHCT1G32

Commit message: Cleanup KiCAD v5 files
Parts:
- J1: value Connector Vertical -> Connector Top
- J2: value Connector Horizontal -> Connector Bot
- renumbered C9 to C1, C1 to C2, C2 to C3, C3 to C4, C10 to C5, C4 to C6, C5 to C7, C6 to C8, C7 to C9
