File: pnp/pcb/ring-light/ringLight.kicad_sch (KiCad schematic)
At the start: 24 parts, among them J1 Connector Top, J2 Connector Bot, U1 74AHCT1G32

Commit message: Move level shifting from ringlight to mobo
Parts:
- removed C5: 100nF, Capacitor_SMD:C_0805_2012Metric, symbol Device:C
- removed R1: 330R, Resistor_SMD:R_0805_2012Metric, symbol Device:R_Small
- removed U1: 74AHCT1G32, Package_TO_SOT_SMD:SOT-353_SC-70-5, symbol 74xGxx:74AHCT1G32
Connections:
- net Data_In_5V is gone; now on net Data: D1.4 (DIN)
- net Data_In_3V3 renamed Data
