File: pnp/pcb/ring-light/ringLight.kicad_pcb (KiCad board)
At the start: 2 copper layers, 40 x 50.2 mm, 33 parts, among them J1 Connector Top, J2 Connector Bot

Commit message: Update PCBs to KiCAD 8
Parts:
- renumbered LOGO to G1
