File: pnp/pcb/ftp/ftp.kicad_pcb (KiCad board)
At the start: 2 copper layers, 75 x 75 mm, 90 parts, among them J1 Conn_01x02_Male

Commit message: Update PCBs to KiCAD 8
Parts:
- renumbered G*** to G1, G*** to G2
