File: pnp/pcb/x-cable-chain-support/x-cable-chain-support.kicad_pcb (KiCad board)
At the start: 2 copper layers, 664 x 44.5 mm, 1 part

Commit message: updates with all current v4 pcbs
Parts:
- added G***: LOGO, index:logo_mask, F.Cu at (66.8, -15.2)
Other:
- board size 664 x 44.5 mm -> 655 x 44.5 mm
