File: pnp/pcb/z-limit/z-limit.kicad_pcb (KiCad board)
At the start: 2 copper layers, 19.8 x 30.3 mm, 8 parts, among them J1 AUX, J2 HEAD_HARNESS, SW1 SW_SPDT

Commit message: updates with all current v4 pcbs
Parts:
- removed kibuzzard-66478BBC: G***, kibuzzard-66478BBC
Other:
- board text added: "REV00"
