File: pnp/pcb/ftp/ftp0402/ftp0402.kicad_pcb (KiCad board)
At the start: 2 copper layers, 75 x 75 mm, 90 parts, among them J1 Conn_01x02_Male

Commit message: tweaks to 0402 ftp
Other:
- board text added: "Functional Test Placement REV00 (0402) 643f8fa docs.opulo.io"
- board text removed: "Functional Test Placement REV01 (0402) <<hash>> docs.opulo.io"
Changed lines of the file:
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@@
 		(tags "resistor")
 		(property "Reference" "R16"
-			(at 0 -1.17 0)
+			(at 0 -1.5 0)
 			(layer "F.SilkS")
 			(effects
@@
 		(tags "resistor")
 		(property "Reference" "R29"
-			(at 0 -1.17 180)
+			(at 0 1.5 180)
 			(layer "F.SilkS")
 			(effects
@@
 		(tags "LED")
 		(property "Reference" "D28"
-			(at 0 -1.17 0)
+			(at 0 -1.5 0)
 			(layer "F.SilkS")
 			(effects
@@
 		(tags "resistor")
 		(property "Reference" "R2"
-			(at 0 -1.17 45)
+			(at 1.69709 0.000015 135)
 			(layer "F.SilkS")
 			(effects
@@
 		(tags "resistor")
 		(property "Reference" "R15"
-			(at 0 -1.17 0)
+			(at 0 -1.5 0)
 			(layer "F.SilkS")
 			(effects
@@
 		(tags "resistor")
 		(property "Reference" "R24"
-			(at 0 -1.17 90)
+			(at 0 -2.25 180)
 			(layer "F.SilkS")
 			(effects
@@
 		(tags "LED")
 		(property "Reference" "D11"
-			(at 0 -1.17 180)
+			(at 0 1.5 180)
 			(layer "F.SilkS")
 			(effects
@@
 		(tags "resistor")
 		(property "Reference" "R3"
-			(at 0 -1.17 0)
+			(at 2.000034 -0.000013 0)
 			(layer "F.SilkS")
 			(effects
@@
 		(tags "resistor")
 		(property "Reference" "R11"
-			(at 0 -1.17 0)
+			(at 0 -1.5 0)
 			(layer "F.SilkS")
 			(effects
@@
 		(tags "resistor")
 		(property "Reference" "R18"
-			(at 0 -1.17 90)
+			(at 0 -2.25 180)
 			(layer "F.SilkS")
 			(effects
@@
 		(tags "LED")
 		(property "Reference" "D15"
-			(at 0 -1.17 180)
+			(at 0 1.5 180)
 			(layer "F.SilkS")
 			(effects
@@
 		(tags "LED")
 		(property "Reference" "D16"
-			(at 0 -1.17 180)
+			(at 0 1.5 180)
 			(layer "F.SilkS")
 			(effects
@@
 		(tags "resistor")
 		(property "Reference" "R32"
-			(at 0 -1.17 180)
+			(at 0 1.5 180)
 			(layer "F.SilkS")
 			(effects
@@
 		(tags "LED")
 		(property "Reference" "D31"
-			(at 0 -1.17 0)
+			(at 0 -1.5 0)
 			(layer "F.SilkS")
 			(effects
@@
 		(tags "LED")
 		(property "Reference" "D19"
-			(at 0 -1.17 270)
+			(at 0 2.25 0)
 			(layer "F.SilkS")
 			(effects
@@
 		(tags "LED")
 		(property "Reference" "D25"
-			(at 0 -1.17 0)
+			(at 0 -1.5 0)
 			(layer "F.SilkS")
 			(effects
@@
 		(tags "resistor")
 		(property "Reference" "R12"
-			(at 0 -1.17 0)
+			(at 0 -1.5 0)
 			(layer "F.SilkS")
 			(effects
@@
 		(tags "resistor")
 		(property "Reference" "R5"
-			(at 0 -1.17 270)
+			(at 1.799987 -0.000034 0)
 			(layer "F.SilkS")
 			(effects
@@
 		(tags "resistor")
 		(property "Reference" "R6"
-			(at 0 -1.17 225)
+			(at 1.838444 -0.000015 315)
 			(layer "F.SilkS")
 			(effects
@@
 		(tags "resistor")
 		(property "Reference" "R23"
-			(at 0 -1.17 90)
+			(at 0 -2.25 180)
 			(layer "F.SilkS")
 			(effects
@@
 		(tags "LED")
 		(property "Reference" "D30"
-			(at 0 -1.17 0)
+			(at 0 -1.5 0)
 			(layer "F.SilkS")
 			(effects
@@
 		(tags "LED")
 		(property "Reference" "D22"
-			(at 0 -1.17 270)
+			(at 0 2.25 0)
 			(layer "F.SilkS")
 			(effects
@@
 		(tags "LED")
 		(property "Reference" "D21"
-			(at 0 -1.17 270)
+			(at 0 2.25 0)
 			(layer "F.SilkS")
 			(effects
@@
 		(tags "LED")
 		(property "Reference" "D32"
-			(at 0 -1.17 0)
+			(at 0 -1.5 0)
 			(layer "F.SilkS")
 			(effects
@@
 		(tags "LED")
 		(property "Reference" "D20"
-			(at 0 -1.17 270)
+			(at 0 2.25 0)
 			(layer "F.SilkS")
 			(effects
@@
 		(tags "resistor")
 		(property "Reference" "R25"
-			(at 0 -1.17 180)
+			(at 0 1.5 180)
 			(layer "F.SilkS")
 			(effects
@@
 		(tags "LED")
 		(property "Reference" "D17"
-			(at 0 -1.17 270)
+			(at 0 2.25 0)
 			(layer "F.SilkS")
 			(effects
@@
 		(tags "LED")
 		(property "Reference" "D26"
-			(at 0 -1.17 0)
+			(at 0 -1.5 0)
 			(layer "F.SilkS")
 			(effects
@@
 		(tags "resistor")
 		(property "Reference" "R4"
-			(at 0 -1.17 315)
+			(at 1.838492 -0.000033 45)
 			(layer "F.SilkS")
 			(effects
@@
 		(tags "LED")
 		(property "Reference" "D3"
-			(at 0 -1.17 270)
+			(at -0.000013 -1.500034 0)
 			(layer "F.SilkS")
 			(effects
@@
 		(tags "LED")
 		(property "Reference" "D23"
-			(at 0 -1.17 270)
+			(at 0 2.25 0)
 			(layer "F.SilkS")
 			(effects
@@
 		(tags "resistor")
 		(property "Reference" "R1"
-			(at 0 -1.17 90)
+			(at 1.600013 0.000034 180)
 			(layer "F.SilkS")
 			(effects
@@
 		(tags "resistor")
 		(property "Reference" "R21"
-			(at 0 -1.17 90)
+			(at 0 -2.25 180)
 			(layer "F.SilkS")
 			(effects
@@
 		(tags "LED")
 		(property "Reference" "D29"
-			(at 0 -1.17 0)
+			(at 0 -1.5 0)
 			(layer "F.SilkS")
 			(effects
@@
 		(tags "resistor")
 		(property "Reference" "R28"
-			(at 0 -1.17 180)
+			(at 0.05 1.5 180)
 			(layer "F.SilkS")
 			(effects
@@
 		(tags "resistor")
 		(property "Reference" "R19"
-			(at 0 -1.17 90)
+			(at 0 -2.25 180)
 			(layer "F.SilkS")
 			(effects
@@
 		(tags "LED")
 		(property "Reference" "D24"
-			(at 0 -1.17 270)
+			(at 0 2.25 0)
 			(layer "F.SilkS")
 			(effects
@@
 		(tags "resistor")
 		(property "Reference" "R17"
-			(at 0 -1.17 90)
+			(at 0 -2.25 180)
 			(layer "F.SilkS")
 			(effects
@@
 		(tags "LED")
 		(property "Reference" "D7"
-			(at 0 -1.17 90)
+			(at 0 -1.599966 180)
 			(layer "F.SilkS")
 			(effects
@@
 		(tags "LED")
 		(property "Reference" "D18"
-			(at 0 -1.17 270)
+			(at 0 2.25 0)
 			(layer "F.SilkS")
 			(effects
@@
 		(tags "resistor")
 		(property "Reference" "R22"
-			(at 0 -1.17 90)
+			(at 0 -2.25 180)
 			(layer "F.SilkS")
 			(effects
@@
 		(tags "LED")
 		(property "Reference" "D12"
-			(at 0 -1.17 180)
+			(at 0 1.5 180)
 			(layer "F.SilkS")
 			(effects
@@
 		(tags "resistor")
 		(property "Reference" "R8"
-			(at 0 -1.17 135)
+			(at 1.697041 0.000033 225)
 			(layer "F.SilkS")
 			(effects
@@
 		(tags "resistor")
 		(property "Reference" "R7"
-			(at 0 -1.17 180)
+			(at 1.999966 0.000013 180)
 			(layer "F.SilkS")
 			(effects
@@
 		(tags "resistor")
 		(property "Reference" "R27"
-			(at 0 -1.17 180)
+			(at 0 1.5 180)
 			(layer "F.SilkS")
 			(effects
@@
 		(tags "resistor")
 		(property "Reference" "R20"
-			(at 0 -1.17 90)
+			(at 0 -2.25 180)
 			(layer "F.SilkS")
 			(effects
@@
 		(tags "resistor")
 		(property "Reference" "R26"
-			(at 0 -1.17 180)
+			(at 0 1.5 180)
 			(layer "F.SilkS")
 			(effects
@@
 		(tags "resistor")
 		(property "Reference" "R31"
-			(at 0 -1.17 180)
+			(at 0 1.5 180)
 			(layer "F.SilkS")
 			(effects
@@
 		(tags "resistor")
 		(property "Reference" "R30"
-			(at 0 -1.17 180)
+			(at 0 1.5 180)
 			(layer "F.SilkS")
 			(effects
@@
 		(tags "LED")
 		(property "Reference" "D27"
-			(at 0 -1.17 0)
+			(at 0 -1.5 0)
 			(layer "F.SilkS")
 			(effects
@@
 		(layer "Edge.Cuts")
 	)
-	(gr_text "Functional Test Placement REV01 (0402)\n<<hash>>\ndocs.opulo.io"
+	(gr_text "Functional Test Placement REV00 (0402)\n643f8fa\ndocs.opulo.io"
 		(at 10 -6.25 0)
 		(layer "F.SilkS")
