File: src/PCB/pi-interface/pi-interface.kicad_sch (KiCad schematic)
At the start: 2 parts, among them J1 PI, J2 MOBO

Commit message: updates readme image, offcenter cam cleanup
Parts:
- added J3: Conn_01x02_Pin, Connector_Molex:Molex_PicoBlade_53261-0271_1x02-1MP_P1.25mm_Horizontal, symbol Connector:Conn_01x02_Pin
Connections:
- net +5V: now also J3.1 (Pin_1)
- net GND: now also J3.2 (Pin_2)
